Commit message: Describe a rover three times the size, and let the old tests object first
Co-Authored-By: Claude Opus 5 <noreply@anthropic.com>

File: cad/urdf/weeding_rover.urdf (robot description, URDF)
Before this commit: robot weeding_rover, 7 links, 6 joints
Links:
- link base_link: mass 0.729560 -> 27.800000; geometry collision box size=0.500 0.340 0.125; collision box size=0.500 0.380 0.155
- link wheel_fl_link: mass 0.075100 -> 1.800000; geometry collision cylinder length=0.090 radius=0.125; visual mesh filename=meshes/wheel.obj
- link wheel_fr_link: mass 0.075100 -> 1.800000; geometry collision cylinder length=0.090 radius=0.125; visual mesh filename=meshes/wheel.obj
- link wheel_rl_link: mass 0.075100 -> 1.800000; geometry collision cylinder length=0.090 radius=0.125; visual mesh filename=meshes/wheel.obj
- link wheel_rr_link: mass 0.075100 -> 1.800000; geometry collision cylinder length=0.090 radius=0.125; visual mesh filename=meshes/wheel.obj
Joints:
- joint camera_down: origin xyz=0 0 0.220 rpy=3.1415926536 0 -1.5707963268 -> xyz=0 0 0.850 rpy=3.1415926536 0 -1.5707963268
- joint camera_front: origin xyz=0.090 0 0.180 rpy=-2.3561944902 0 -1.5707963268 -> xyz=0 0 0.850 rpy=-2.4434609528 0 -1.5707963268
- joint wheel_fl: limit effort=0.4903 velocity=5.7714 -> effort=10.0 velocity=2.616; origin xyz=0.060 0.060 0.035 rpy=0 0 0 -> xyz=0.200 0.215 0.125 rpy=0 0 0
- joint wheel_fr: limit effort=0.4903 velocity=5.7714 -> effort=10.0 velocity=2.616; origin xyz=0.060 -0.060 0.035 rpy=0 0 0 -> xyz=0.200 -0.215 0.125 rpy=0 0 0
- joint wheel_rl: limit effort=0.4903 velocity=5.7714 -> effort=10.0 velocity=2.616; origin xyz=-0.060 0.060 0.035 rpy=0 0 0 -> xyz=-0.200 0.215 0.125 rpy=0 0 0
- joint wheel_rr: limit effort=0.4903 velocity=5.7714 -> effort=10.0 velocity=2.616; origin xyz=-0.060 -0.060 0.035 rpy=0 0 0 -> xyz=-0.200 -0.215 0.125 rpy=0 0 0
